File: LTC1779_CV Controlled_Non-Inv.kicad_pcb (KiCad board)
At the start: 2 copper layers, 34 x 39 mm, 31 parts, among them J1 CV_In_1, J2 SET, J3 DIVIDE, J4 To Board, J5 CV_Mix_1, J6 CV_In_1, J7 CV_Mix_2, U1 MCP6002-xSN, U2 MCP6002-xSN, U3 LTC1799

Commit message: added a logo
Parts:
- added G***: LOGO, Library:voltagecontrolledclock(xs), F.Cu at (138.4, 59.9)
- added G***: LOGO, Library:voltagecontrolledclock, B.Cu at (139.1, 72.1)
- C3: value 0.1uF -> 100nF
