File: LTC1779_CV Controlled_Non-Inv.kicad_sch (KiCad schematic)
At the start: 30 parts, among them J1 CV_In_1, J2 SET, J3 DIVIDE, J4 To Board, J5 CV_Mix_1, J6 CV_In_1, J7 CV_Mix_2, U1 MCP6002-xSN, U2 MCP6002-xSN, U3 LTC1799

Commit message: added a logo
Parts:
- C3: value 0.1uF -> 100nF
